Commit message: camera URDF

File: src/cuscobot_core/urdf/camera.xacro (robot description, xacro)
@@ -1,4 +1,5 @@
 <?xml version="1.0"?>
 <robot xmlns:xacro="http://www.ros.org/wiki/xacro" >
+    <xacro:property name="half_pi_const" value="1.570796" />
     <joint name="camera_joint" type="fixed">
         <parent link="base_link"/>
@@ -17,5 +18,6 @@
         <parent link="camera_link"/>
         <child link="camera_optical_link"/>
-        <origin xyz="0 0 0" rpy="{-half_pi_const} 0 {-half_pi_const}"/>
+        <origin xyz="0 0 0" rpy="${-half_pi_const} 0 ${-half_pi_const}"/>
     </joint>
+    <link name="camera_optical_link"></link>
 </robot>

Commit message: YOLO and VO tests

File: src/cuscobot_core/urdf/camera.xacro (robot description, xacro)
@@ -18,5 +18,6 @@
         <parent link="camera_link"/>
         <child link="camera_optical_link"/>
-        <origin xyz="0 0 0" rpy="${-half_pi_const} 0 ${-half_pi_const}"/>
+        <origin xyz="0 0 0" rpy="0 0 0"/>
+        <!-- <origin xyz="0 0 0" rpy="${-half_pi_const} 0 ${-half_pi_const}"/> -->
     </joint>
     <link name="camera_optical_link"></link>
